File: display/display.kicad_pcb (KiCad board)
At the start: 2 copper layers, 253 x 44 mm, 0 parts

Commit message: display.kicad_pcb, display.zip und 2 weitere dateien aktualisiert...
Routing:
- added copper zone on B.Cu, net (none)
Other:
- outline, holes or cut-outs redrawn
Changed lines of the file:
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@@
 	)
 	(net 0 "")
-	(gr_circle
-		(center 267 102.5)
-		(end 267 103)
-		(stroke
-			(width 0.2)
-			(type default)
-		)
-		(fill no)
-		(layer "F.Cu")
-	)
-	(gr_circle
-		(center 32 102.5)
-		(end 32 103)
-		(stroke
-			(width 0.2)
-			(type default)
-		)
-		(fill no)
-		(layer "F.Cu")
-	)
-	(gr_circle
-		(center 267 70.5)
-		(end 267 71)
-		(stroke
-			(width 0.2)
-			(type default)
-		)
-		(fill no)
-		(layer "F.Cu")
-	)
-	(gr_circle
-		(center 32 70.5)
-		(end 32 71)
-		(stroke
-			(width 0.2)
-			(type default)
-		)
-		(fill no)
-		(layer "F.Cu")
-	)
 	(gr_arc
 		(start 94.5 77.5)
@@
 	)
 	(gr_circle
-		(center 218.5 68.5)
-		(end 220 68.5)
+		(center 219 68.5)
+		(end 220.5 68.5)
 		(stroke
 			(width 0.2)
@@
 	)
 	(gr_circle
-		(center 218.5 104.5)
-		(end 220 104.5)
+		(center 219 104.5)
+		(end 220.5 104.5)
 		(stroke
 			(width 0.2)
@@
 	)
 	(gr_circle
-		(center 80 68.5)
-		(end 81.5 68.5)
+		(center 79.5 68.5)
+		(end 81 68.5)
 		(stroke
 			(width 0.2)
@@
 	)
 	(gr_circle
-		(center 80 104.5)
-		(end 81.5 104.5)
+		(center 79.5 104.5)
+		(end 81 104.5)
 		(stroke
 			(width 0.2)
@@
 		)
 	)
+	(zone
+		(net 0)
+		(net_name "")
+		(layer "B.Cu")
+		(hatch edge 0.5)
+		(connect_pads
+			(clearance 0.5)
+		)
+		(min_thickness 0.25)
+		(filled_areas_thickness no)
+		(fill yes
+			(thermal_gap 0.5)
+			(thermal_bridge_width 0.5)
+			(island_removal_mode 1)
+			(island_area_min 10)
+		)
+		(polygon
+			(pts
+				(xy 18 55) (xy 279.5 58) (xy 280.5 125) (xy 19.5 121)
+			)
+		)
+	)
