File: tl-sg108e/tl-sg108e.kicad_pcb (KiCad board)
At the start: 2 copper layers, 215 x 44 mm, 0 parts

Commit message: display.kicad_pcb, display.zip und 2 weitere dateien aktualisiert...
Changed lines of the file:
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@@
 	(net 0 "")
 	(gr_line
-		(start 229.5 89.5)
-		(end 77.5 89.5)
+		(start 77.5 89.5)
+		(end 229.5 89.5)
+		(stroke
+			(width 0.2)
+			(type solid)
+		)
+		(layer "Edge.Cuts")
+	)
+	(gr_line
+		(start 232.5 92.5)
+		(end 232.5 112.5)
 		(stroke
 			(width 0.2)
@@
 		(mid 75.37868 90.37868)
 		(end 77.5 89.5)
-		(stroke
-			(width 0.2)
-			(type solid)
-		)
-		(layer "Edge.Cuts")
-	)
-	(gr_line
-		(start 74.5 112.5)
-		(end 74.5 92.5)
 		(stroke
 			(width 0.2)
@@
 	)
 	(gr_line
-		(start 232.5 112.5)
-		(end 232.5 92.5)
+		(start 74.5 112.5)
+		(end 74.5 92.5)
 		(stroke
 			(width 0.2)
